File: BlinkenPDS.kicad_sch (KiCad schematic)
At the start: 256 parts, among them CN1 PDS_LB_MALE, CN2 PDS_PT_FEMALE RA, CN3 PDS_PT_FEMALE ST, U1 74HC14D, U10 74HC14D, U11 74HC14D, U12 74HC14D, U13 74HC14D, U14 74HC14D, U15 74HC14D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

Commit message: remove PFW, add CACHE, updated production files
Parts:
- removed D67: C, SockeBooster:LED_0603_1608Metric_Label, symbol Device:LED
- removed R68: 510, SockeBooster:R_0402_1005Metric_NoLabel, symbol Device:R
- U18: now not fitted; now left out of the parts list
Connections:
- net C16M: no longer U1.1 (I1)
- net GND: now also U1.1 (I1); no longer CN1.B2 (GND), CN2.B2 (GND), CN3.B2 (GND)
- net RESA1: now also U13.13 (I6)
- removed net PFW: CN1.C1 (PFW), CN2.C1 (PFW), CN3.C1 (PFW), U13.9 (I4)
- new net CACHE: CN1.B2 (CACHE), CN2.B2 (CACHE), CN3.B2 (CACHE), U13.9 (I4)
- no-connect marks 0 -> 3
